File: KiCAD Stuff/Capstone/Capstone.kicad_sch (KiCad schematic)
At the start: 31 parts, among them J1 -EEG_INPUT, J2 +EEG_INPUT, U1 INA819, U2 TPS61094, U3 TLV9102, U4 TC1044, U5 TLV9102

Commit message: Added a new project that takes TLV9102 as an 8-pin SOIC
Parts:
- added J3: +3.3V, symbol Connector:Conn_01x01_Socket
- added J4: GND, symbol Connector:Conn_01x01_Socket
- R4: value 150k -> 4.75k
Connections:
- net +3.3V: now also J3.1 (Pin_1)
- net GND: now also J4.1 (Pin_1)
Changed lines of the file:
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@@
   (junction (at 121.92 147.32) (diameter 0) (color 0 0 0 0)
   )
+  (junction (at 129.54 118.11) (diameter 0) (color 0 0 0 0)
+  )
   (junction (at 77.47 124.46) (diameter 0) (color 0 0 0 0)
   )
@@
     (stroke (width 0) (type default))
   )
+  (wire (pts (xy 129.54 118.11) (xy 135.89 118.11))
+    (stroke (width 0) (type default))
+  )
   (wire (pts (xy 152.4 43.18) (xy 156.21 43.18))
     (stroke (width 0) (type default))
@@
     (stroke (width 0) (type default))
   )
-  (wire (pts (xy 121.92 118.11) (xy 135.89 118.11))
+  (wire (pts (xy 121.92 118.11) (xy 129.54 118.11))
     (stroke (width 0) (type default))
   )
@@
     )
   )
+  (symbol (lib_id "Connector:Conn_01x01_Socket") (at 129.54 113.03 270) (mirror x) (unit 1)
+    (in_bom yes) (on_board yes) (dnp no)
+    (property "Reference" "J3" (at 130.81 107.95 90)
+      (effects (font (size 1.27 1.27)) (justify right))
+    )
+    (property "Value" "+3.3V" (at 130.81 110.49 90)
+      (effects (font (size 1.27 1.27)) (justify right))
+    )
+    (property "Footprint" "" (at 129.54 113.03 0)
+      (effects (font (size 1.27 1.27)) hide)
+    )
+    (property "Datasheet" "~" (at 129.54 113.03 0)
+      (effects (font (size 1.27 1.27)) hide)
+    )
+    (pin "1")
+    (instances
+      (project "Capstone"
+        (path "/14ccd594-9acb-4c8c-856d-2255d639ffb5"
+          (reference "J3") (unit 1)
+        )
+      )
+      (project "Capstone"
+        (path "/dd9861b4-b57a-4b4e-bd42-9d4b17c05a17"
+          (reference "J1") (unit 1)
+        )
+      )
+    )
+  )
   (symbol (lib_id "Device:C") (at 53.34 133.35 0) (unit 1)
     (in_bom yes) (on_board yes) (dnp no) (fields_autoplaced)
@@
       (effects (font (size 1.27 1.27)) (justify left))
     )
-    (property "Value" "150k" (at 71.12 134.62 0)
+    (property "Value" "4.75k" (at 71.12 134.62 0)
       (effects (font (size 1.27 1.27)) (justify left))
     )
@@
         )
       )
+    )
+  )
+  (symbol (lib_id "Connector:Conn_01x01_Socket") (at 121.92 152.4 90) (mirror x) (unit 1)
+    (in_bom yes) (on_board yes) (dnp no)
+    (property "Reference" "J4" (at 120.65 157.48 90)
+      (effects (font (size 1.27 1.27)) (justify right))
+    )
+    (property "Value" "GND" (at 120.65 154.94 90)
+      (effects (font (size 1.27 1.27)) (justify right))
+    )
+    (property "Footprint" "" (at 121.92 152.4 0)
+      (effects (font (size 1.27 1.27)) hide)
+    )
+    (property "Datasheet" "~" (at 121.92 152.4 0)
+      (effects (font (size 1.27 1.27)) hide)
+    )
+    (pin "1")
+    (instances
+      (project "Capstone"
+        (path "/14ccd594-9acb-4c8c-856d-2255d639ffb5"
+          (reference "J4") (unit 1)
+        )
+      )
+      (project "Capstone"
+        (path "/dd9861b4-b57a-4b4e-bd42-9d4b17c05a17"
+          (reference "J1") (unit 1)
+        )
+      )
