File: PCB_design_files/P1.2/P1.2.kicad_sch (KiCad schematic)
At the start: 48 parts, among them J1 EEG_IN-, J10 BAT+, J11 BOOST, J2 EEG_IN+, J3 +3.3V, J4 GND, J5 -3V3, J6 EEG_INPUT, J7 STAGE_1_OUT, J8 STAGE_2_OUT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

Commit message: Added offset
Parts:
- added C11: 10uF, symbol Device:C
- added R22, R23, R24, R25, R27: 100k, symbol Device:R
- added R26: 100k, Potentiometer_THT:Potentiometer_Bourns_3296W_Vertical, symbol Device:R_Potentiometer
- added R28: 10k, symbol Device:R
- R12, R16, R19: value 5k -> 5.1k
Connections:
- net +3.3V: now also R26.2
- net Conditioned_EEG: now also R23.2, R24.1, R27.2, R28.2; no longer C10.1, C8.1, C9.1, R17.2, R21.1, R8.2
- net GND: now also R22.2, R25.2
- new net: R23.1, R26.1, R27.1
- new net: C10.1, C11.1, C8.1, C9.1, R17.2, R21.1, R8.2
- new net: C11.2, R22.1, R28.1
- new net: R24.2, R25.1

Commit message: Updated schematic
Parts:
- added D1: LED, symbol Device:LED
- added J12, J13: Conn_01x06_Pin, symbol Connector:Conn_01x06_Pin
- added R29: 7k, symbol Device:R
- added R30: 50k, symbol Device:R
- added SW1: DS04-254-1S-01BK, symbol Switch:SW_DIP_x01
- added U5: ~, symbol My_Library:TLC1059
Connections:
- net +3.3V: now also J13.6 (Pin_6), U5.5 (SA), U5.6 (V+), U5.9 (50/100/HOLD)
- net -3V3: now also U5.10 (V-)
- net BAT+: now also SW1.1; no longer BT1.1 (+), C1.1, L1.1, U2.2 (MODE), U2.3 (EN), U2.4 (VIN), U2.6 (SUP)
- net Conditioned_EEG: now also J13.2 (Pin_2), R29.2, U5.2 (N/AP/HP); no longer R23.2, R24.1, R27.2, R28.2
- net GND: now also J12.1 (Pin_1), U5.11 (AGND), U5.7 (LSh)
- new net: R23.2, R24.1, R27.2, R28.2, R29.1, R30.1, U5.3 (INV1)
- new net: R30.2, U5.1 (BP)
- new net: BT1.1 (+), C1.1, D1.1 (K), L1.1, U2.2 (MODE), U2.3 (EN), U2.4 (VIN), U2.6 (SUP)
- new net: D1.2 (A), SW1.2
- new net: U5.14 (LP), U5.4 (S1)
- new net +5V: J13.1 (Pin_1)
- new net CLK: J12.3 (Pin_3), U5.8 (CLK)
Other:
- moved on the sheet: BT1, C1, C10, C11, C2, C3, C4, C5, C6, C7, C8, C9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

Commit message: Updated schematic based on Alberts latest changes
Parts:
- added J14: STAGE_3_OUT, TestPoint:TestPoint_Loop_D2.50mm_Drill1.0mm, symbol Connector:Conn_01x01_Socket
- added R31: 15, Resistor_THT:R_Axial_DIN0207_L6.3mm_D2.5mm_P10.16mm_Horizontal, symbol Device:R
- C11: footprint (none) -> Capacitor_THT:CP_Radial_D5.0mm_P2.50mm
- D1: value LED -> LED_PWR; footprint (none) -> LED_THT:LED_D10.0mm
- J12, J13: footprint (none) -> Connector_PinSocket_2.54mm:PinSocket_1x06_P2.54mm_Vertical
- J9: value STAGE_3_OUT -> CONDITIONED
- R14, R15, R16, R17, R18, R19, R20, R22, R23, R24, R25, R27, R28, R29, R30: footprint (none) -> Resistor_THT:R_Axial_DIN0207_L6.3mm_D2.5mm_P10.16mm_Horizontal
- U1, U3: footprint 1-2199298-2:CONN8_1-2199298-2_TEC -> Package_DIP:DIP-8_W7.62mm_Socket_LongPads
- U5: value ~ -> LTC1059CS#PBF; footprint (none) -> Package_DIP:DIP-14_W7.62mm_LongPads
Connections:
- net BAT+: now also BT1.1 (+)
- net GND: now also D1.1 (K)
- net STAGE_3_OUT: now reaches R23.2, R24.1, R27.2, R28.2, R29.1, R30.1, U5.3 (INV1)
- net STAGE_3_OUT: now also J14.1 (Pin_1)
- net at C1.1, L1.1, U2.2 (MODE)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: now also SW1.2, R31.1; no longer BT1.1 (+), D1.1 (K)
- net at D1.2 (A): now also R31.2; no longer SW1.2
Other:
- moved on the sheet: C1, C3, C5, C6, J11, J7, J8, J9, L1, R29, R30, R4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

Commit message: Added footprint for power switch
Parts:
- SW1: footprint (none) -> DS04_254_1S_01BK:SW_DS04-254-1S-01BK
Changed lines of the file:
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@@
     (fill (type none))
-  )
-  (text_box "add switch footprint\n"
-    (at 73.66 144.78 0) (size 22.86 5.08)
-    (stroke (width 0) (type default))
-    (fill (type color) (color 255 215 209 1))
-    (effects (font (size 1.27 1.27)) (justify left top))
   )
   (text_box "Legend:\nJ12:     J13:\n1 - GND  1 - 5V\n2 - D2   2 - A0\n3 - D3   3 - A1\n4 - D4   4 - A2\n5 - D5   5 - A3\n6 - GND  6 - VIN\nAlbert - I couldn't rename the pins on the headers so I just made this instead"
@@
       (effects (font (size 1.27 1.27)))
     )
-    (property "Footprint" "" (at 64.77 158.75 0)
-      (effects (font (size 1.27 1.27)) hide)
-    )
+    (property "Footprint" "DS04_254_1S_01BK:SW_DS04-254-1S-01BK" (at 64.77 158.75 0)
+      (effects (font (size 1.27 1.27)) hide)
+    )

Commit message: Minor schematic changes
Parts:
- added H1, H2, H3, H4: MountingHole, MountingHole:MountingHole_3.2mm_M3, symbol Mechanical:MountingHole
Other:
- note added: "Mechanical standoffs"
- moved on the sheet: C11, R22, R23, R24, R25, R26, R27, R28, R29, R30, U5

Commit message: Updated resistor values
Parts:
- removed R14, R15, R20: 1k, Resistor_THT:R_Axial_DIN0207_L6.3mm_D2.5mm_P10.16mm_Horizontal, symbol Device:R
- removed R16, R19: 5.1k, Resistor_THT:R_Axial_DIN0207_L6.3mm_D2.5mm_P10.16mm_Horizontal, symbol Device:R
- removed R17, R25, R27: 100k, Resistor_THT:R_Axial_DIN0207_L6.3mm_D2.5mm_P10.16mm_Horizontal, symbol Device:R
- removed R18: 3k, Resistor_THT:R_Axial_DIN0207_L6.3mm_D2.5mm_P10.16mm_Horizontal, symbol Device:R
- D1: footprint LED_THT:LED_D10.0mm -> LED_THT:LED_D5.0mm
- R10: value 100 -> 604
- R11: value 10k -> 16k
- R12: value 5.1k -> 2.49k
- R2: value 5.1k -> 8.2k
- R23, R8: value 100k -> 49.9k
- R24: value 100k -> 200k
- R29: value 7k -> 6.98k
- R30: value 50k -> 49.9k
- R31: value 15 -> 10k
Connections:
- net GND: now also R24.2
- net at R2.1: now also U1.2 (RG)
- net at R11.2: now also C7.2, U3.5 (IN2+)
- net at C4.2, R9.1: now also R10.1
Other:
- moved on the sheet: R10, R2, R22, R24

Commit message: Changes
Parts:
- removed R22: 100k, Resistor_THT:R_Axial_DIN0207_L6.3mm_D2.5mm_P10.16mm_Horizontal, symbol Device:R
- removed R26: 100k, Potentiometer_THT:Potentiometer_Bourns_3296W_Vertical, symbol Device:R_Potentiometer
- removed R29: 6.98k, Resistor_THT:R_Axial_DIN0207_L6.3mm_D2.5mm_P10.16mm_Horizontal, symbol Device:R
- removed R30: 49.9k, Resistor_THT:R_Axial_DIN0207_L6.3mm_D2.5mm_P10.16mm_Horizontal, symbol Device:R
- removed U5: LTC1059CS#PBF, Package_DIP:DIP-14_W7.62mm_LongPads, symbol My_Library:TLC1059
- R23: value 49.9k -> 200k
Connections:
- net +3.3V: now also R23.1
- net Conditioned_EEG: now also C11.2, R23.2, R24.1
- net STAGE_3_OUT: no longer R23.2, R24.1, R28.2
- net at R28.1: now also C10.1, C8.1, C9.1, R21.1, R8.2; no longer C11.2
- net CLK: no longer names the net of J12.3 (Pin_3)
- new net: C11.1, R28.2
Other:
- moved on the sheet: C11, R23, R24, R28
