File: PCB_design_files/P2.0/P2.0.kicad_sch (KiCad schematic)
At the start: 54 parts, among them J1 EEG_IN, J3 SWD, U1 INA819IDRGR, U3 TPS61094, U5 NRF52832-QFAA-R, X1 32MHz

Commit message: Footprint
Parts:
- removed U4: ~, symbol TPS60400DBVR:TPS60400DBVR
- added U4: TPS60400, symbol Amplifier_Current:AD8211
- R17: value ?150k -> 100k
- R6: value ?100k -> 100k
Connections:
- net +3V3: now also U4.1 (IN)
- net -3V3: now also U4.5 (OUT)
- net GND: now also U4.2 (GND)
- net at C10.1: now also U4.3 (CFLY+)
- net at C10.2: now also U4.4 (CFLY-)
Changed lines of the file:
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@@
   (junction (at 133.35 39.37) (diameter 0) (color 0 0 0 0)
   )
-  (junction (at 312.42 119.38) (diameter 0) (color 0 0 0 0)
-  )
   (junction (at 232.41 71.12) (diameter 0) (color 0 0 0 0)
   )
@@
     (stroke (width 0) (type default))
   )
-  (wire (pts (xy 312.42 119.38) (xy 312.42 102.87))
-    (stroke (width 0) (type default))
-  )
   (wire (pts (xy 208.28 67.31) (xy 208.28 54.61))
     (stroke (width 0) (type default))
@@
     (stroke (width 0) (type default))
   )
+  (wire (pts (xy 303.53 104.14) (xy 303.53 105.41))
+    (stroke (width 0) (type default))
+  )
   (wire (pts (xy 212.09 125.73) (xy 237.49 125.73))
     (stroke (width 0) (type default))
@@
     (stroke (width 0) (type default))
   )
-  (wire (pts (xy 295.91 149.86) (xy 302.26 149.86))
+  (wire (pts (xy 290.83 149.86) (xy 302.26 149.86))
     (stroke (width 0) (type default))
   )
@@
     (stroke (width 0) (type default))
   )
-  (wire (pts (xy 312.42 129.54) (xy 312.42 119.38))
-    (stroke (width 0) (type default))
-  )
   (wire (pts (xy 270.51 137.16) (xy 270.51 140.97))
     (stroke (width 0) (type default))
@@
     (stroke (width 0) (type default))
   )
-  (wire (pts (xy 306.07 142.24) (xy 306.07 132.08))
+  (wire (pts (xy 306.07 142.24) (xy 306.07 133.35))
+    (stroke (width 0) (type default))
+  )
+  (wire (pts (xy 313.69 129.54) (xy 318.77 129.54))
     (stroke (width 0) (type default))
   )
@@
     (stroke (width 0) (type default))
   )
+  (wire (pts (xy 299.72 125.73) (xy 298.45 125.73))
+    (stroke (width 0) (type default))
+  )
   (wire (pts (xy 162.56 39.37) (xy 162.56 31.75))
     (stroke (width 0) (type default))
@@
     (stroke (width 0) (type default))
   )
+  (wire (pts (xy 299.72 132.08) (xy 299.72 125.73))
+    (stroke (width 0) (type default))
+  )
   (wire (pts (xy 203.2 25.4) (xy 203.2 35.56))
     (stroke (width 0) (type default))
@@
     (stroke (width 0) (type default))
   )
-  (wire (pts (xy 312.42 129.54) (xy 318.77 129.54))
+  (wire (pts (xy 293.37 115.57) (xy 293.37 129.54))
     (stroke (width 0) (type default))
   )
@@
     (stroke (width 0) (type default))
   )
-  (wire (pts (xy 306.07 132.08) (xy 304.8 132.08))
+  (wire (pts (xy 306.07 133.35) (xy 308.61 133.35))
     (stroke (width 0) (type default))
   )
@@
     (stroke (width 0) (type default))
   )
-  (wire (pts (xy 302.26 132.08) (xy 302.26 137.16))
-    (stroke (width 0) (type default))
-  )
   (wire (pts (xy 266.7 121.92) (xy 270.51 121.92))
     (stroke (width 0) (type default))
@@
     (stroke (width 0) (type default))
   )
-  (wire (pts (xy 295.91 137.16) (xy 295.91 149.86))
-    (stroke (width 0) (type default))
-  )
   (wire (pts (xy 106.68 109.22) (xy 109.22 109.22))
     (stroke (width 0) (type default))
@@
     (stroke (width 0) (type default))
   )
+  (wire (pts (xy 313.69 110.49) (xy 313.69 129.54))
+    (stroke (width 0) (type default))
+  )
   (wire (pts (xy 250.19 71.12) (xy 250.19 81.28))
     (stroke (width 0) (type default))
@@
     (stroke (width 0) (type default))
   )
+  (wire (pts (xy 290.83 149.86) (xy 290.83 104.14))
+    (stroke (width 0) (type default))
+  )
   (wire (pts (xy 48.26 53.34) (xy 31.75 53.34))
     (stroke (width 0) (type default))
@@
     (stroke (width 0) (type default))
   )
+  (wire (pts (xy 290.83 104.14) (xy 303.53 104.14))
+    (stroke (width 0) (type default))
+  )
   (wire (pts (xy 189.23 142.24) (xy 189.23 152.4))
     (stroke (width 0) (type default))
@@
     (stroke (width 0) (type default))
   )
-  (wire (pts (xy 302.26 102.87) (xy 292.1 102.87))
-    (stroke (width 0) (type default))
-  )
-  (wire (pts (xy 292.1 102.87) (xy 292.1 129.54))
-    (stroke (width 0) (type default))
-  )
   (wire (pts (xy 144.78 29.21) (xy 144.78 34.29))
     (stroke (width 0) (type default))
@@
     (stroke (width 0) (type default))
   )
-  (wire (pts (xy 302.26 137.16) (xy 295.91 137.16))
-    (stroke (width 0) (type default))
-  )
   (wire (pts (xy 38.1 40.64) (xy 66.04 40.64))
     (stroke (width 0) (type default))
   )
-  (wire (pts (xy 304.8 102.87) (xy 312.42 102.87))
-    (stroke (width 0) (type default))
-  )
   (wire (pts (xy 121.285 185.42) (xy 135.255 185.42))
     (stroke (width 0) (type default))
@@
     (stroke (width 0) (type default))
   )
+  (wire (pts (xy 308.61 125.73) (xy 308.61 133.35))
+    (stroke (width 0) (type default))
+  )
   (wire (pts (xy 266.7 129.54) (xy 278.13 129.54))
     (stroke (width 0) (type default))
@@
     (stroke (width 0) (type default))
   )
-  (wire (pts (xy 278.13 129.54) (xy 292.1 129.54))
+  (wire (pts (xy 278.13 129.54) (xy 293.37 129.54))
     (stroke (width 0) (type default))
   )
@@
       (effects (font (size 1.27 1.27)) (justify left))
     )
-    (property "Value" "?100k" (at 135.89 35.56 0)
+    (property "Value" "100k" (at 135.89 35.56 0)
       (effects (font (size 1.27 1.27)) (justify left))
     )
@@
       (effects (font (size 1.27 1.27)) (justify left))
     )
-    (property "Value" "?150k" (at 280.67 36.83 0)
+    (property "Value" "100k" (at 280.67 36.83 0)
       (effects (font (size 1.27 1.27)) (justify left))
     )
@@
         (path "/cc4d5c34-4776-48f9-a8ce-15f2c8e358ac"
           (reference "R12") (unit 1)
+        )
+      )
+    )
+  )
+  (symbol (lib_id "Amplifier_Current:AD8211") (at 303.53 115.57 180) (unit 1)
+    (in_bom yes) (on_board yes) (dnp no) (fields_autoplaced)
+    (property "Reference" "U4" (at 290.83 119.2179 0)
+      (effects (font (size 1.27 1.27)))
+    )
+    (property "Value" "TPS60400" (at 290.83 116.6779 0)
+      (effects (font (size 1.27 1.27)))
+    )
+    (property "Footprint" "" (at 303.53 115.57 0)
+      (effects (font (size 1.27 1.27)) hide)
+    )
+    (property "Datasheet" "" (at 287.02 97.79 0)
+      (effects (font (size 1.27 1.27)) hide)
+    )
+    (pin "3")
+    (pin "4")
+    (pin "5")
+    (pin "1")
+    (pin "2")
+    (instances
+      (project "P2.0"
+        (path "/cc4d5c34-4776-48f9-a8ce-15f2c8e358ac"
+          (reference "U4") (unit 1)
         )
       )
@@
         )
       )
-    )
-  )
-  (symbol (lib_id "TPS60400DBVR:TPS60400DBVR") (at 309.88 110.49 270) (unit 1)
-    (in_bom yes) (on_board yes) (dnp no)
-    (property "Reference" "U4" (at 313.69 121.92 0)
-      (effects (font (size 1.27 1.27)) (justify left))
-    )
-    (property "Value" "~" (at 309.88 110.49 0)
-      (effects (font (size 1.27 1.27)))
-    )
-    (property "Footprint" "" (at 309.88 110.49 0)
-      (effects (font (size 1.27 1.27)) hide)
-    )
-    (property "Datasheet" "" (at 309.88 110.49 0)
-      (effects (font (size 1.27 1.27)) hide)
-    )
-    (pin "3")
-    (pin "4")
-    (pin "5")
-    (pin "2")
-    (pin "1")
-    (pin "8")
-    (pin "6")
-    (pin "7")
-    (pin "9")
-    (pin "10")
-    (instances
-      (project "P2.0"
-        (path "/cc4d5c34-4776-48f9-a8ce-15f2c8e358ac"
-          (reference "U4") (unit 1)
-        )
-      )
