File: PCB_design_files/P2.0/P2.0.kicad_sch (KiCad schematic)
At the start: 58 parts, among them J1 EEG_IN, J2 Conn_02x03_Counter_Clockwise, U1 INA819IDRGR, U2 TLV9102IDSGR, U3 TPS61094, U4 TPS60400, U5 NRF52832-QFAA-R, Y1 32MHz

Commit message: Generated assembly files and rearranged manufacturing files
Parts:
- AE1: Manufacturer (none) -> Johanson Technology Inc.; Part Number (none) -> 2450AT18B0100001E
- BT1, J1: Manufacturer (none) -> n/a; Part Number (none) -> n/a
- D1: Manufacturer (none) -> Würth Elektronik; Part Number (none) -> 150060VS75000
- J2: Manufacturer (none) -> Amphenol ICC (FCI); Part Number (none) -> 20021121-00006C4LF
- U5: Manufacturer (none) -> Nordic Semiconductor ASA; Part Number (none) -> NRF52832-QFAA-R
- Y1: Manufacturer (none) -> ECS Inc.; Part Number (none) -> ECS-320-8-37CKM
Changed lines of the file:
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@@
       (effects (font (size 1.27 1.27) italic) hide)
     )
-    (property "Description" "" (at 47.625 125.73 0)
-      (effects (font (size 1.27 1.27)) hide)
-    )
-    (property "Manufacturer" "" (at 47.625 125.73 0)
-      (effects (font (size 1.27 1.27)) hide)
-    )
-    (property "Part Number" "" (at 47.625 125.73 0)
+    (property "Description" "IC RF TXRX+MCU BLUETOOTH 48VFQFN" (at 47.625 125.73 0)
+      (effects (font (size 1.27 1.27)) hide)
+    )
+    (property "Manufacturer" "Nordic Semiconductor ASA" (at 47.625 125.73 0)
+      (effects (font (size 1.27 1.27)) hide)
+    )
+    (property "Part Number" "NRF52832-QFAA-R" (at 47.625 125.73 0)
       (effects (font (size 1.27 1.27)) hide)
     )
@@
       (effects (font (size 1.27 1.27)) hide)
     )
-    (property "Description" "" (at 24.13 48.26 0)
-      (effects (font (size 1.27 1.27)) hide)
-    )
-    (property "Manufacturer" "" (at 24.13 48.26 0)
-      (effects (font (size 1.27 1.27)) hide)
-    )
-    (property "Part Number" "" (at 24.13 48.26 0)
+    (property "Description" "No Part" (at 24.13 48.26 0)
+      (effects (font (size 1.27 1.27)) hide)
+    )
+    (property "Manufacturer" "n/a" (at 24.13 48.26 0)
+      (effects (font (size 1.27 1.27)) hide)
+    )
+    (property "Part Number" "n/a" (at 24.13 48.26 0)
       (effects (font (size 1.27 1.27)) hide)
     )
@@
       (effects (font (size 1.27 1.27)) hide)
     )
-    (property "Description" "" (at 129.54 132.08 0)
-      (effects (font (size 1.27 1.27)) hide)
-    )
-    (property "Manufacturer" "" (at 129.54 132.08 0)
-      (effects (font (size 1.27 1.27)) hide)
-    )
-    (property "Part Number" "" (at 129.54 132.08 0)
+    (property "Description" "CRYSTAL 32.0000MHZ 8PF SMD" (at 129.54 132.08 0)
+      (effects (font (size 1.27 1.27)) hide)
+    )
+    (property "Manufacturer" "ECS Inc." (at 129.54 132.08 0)
+      (effects (font (size 1.27 1.27)) hide)
+    )
+    (property "Part Number" "ECS-320-8-37CKM" (at 129.54 132.08 0)
       (effects (font (size 1.27 1.27)) hide)
     )
@@
       (effects (font (size 1.27 1.27)) hide)
     )
-    (property "Description" "" (at 184.15 139.7 0)
-      (effects (font (size 1.27 1.27)) hide)
-    )
-    (property "Manufacturer" "" (at 184.15 139.7 0)
-      (effects (font (size 1.27 1.27)) hide)
-    )
-    (property "Part Number" "" (at 184.15 139.7 0)
+    (property "Description" "No Part" (at 184.15 139.7 0)
+      (effects (font (size 1.27 1.27)) hide)
+    )
+    (property "Manufacturer" "n/a" (at 184.15 139.7 0)
+      (effects (font (size 1.27 1.27)) hide)
+    )
+    (property "Part Number" "n/a" (at 184.15 139.7 0)
       (effects (font (size 1.27 1.27)) hide)
     )
@@
       (effects (font (size 1.27 1.27)) hide)
     )
-    (property "Description" "" (at 150.495 176.53 0)
-      (effects (font (size 1.27 1.27)) hide)
-    )
-    (property "Manufacturer" "" (at 150.495 176.53 0)
-      (effects (font (size 1.27 1.27)) hide)
-    )
-    (property "Part Number" "" (at 150.495 176.53 0)
+    (property "Description" "RF ANT 2.4GHZ CHIP SOLDER SMD" (at 150.495 176.53 0)
+      (effects (font (size 1.27 1.27)) hide)
+    )
+    (property "Manufacturer" "Johanson Technology Inc." (at 150.495 176.53 0)
+      (effects (font (size 1.27 1.27)) hide)
+    )
+    (property "Part Number" "2450AT18B0100001E" (at 150.495 176.53 0)
       (effects (font (size 1.27 1.27)) hide)
     )
@@
       (effects (font (size 1.27 1.27)) hide)
     )
-    (property "Description" "" (at 330.2 134.62 0)
-      (effects (font (size 1.27 1.27)) hide)
-    )
-    (property "Manufacturer" "" (at 330.2 134.62 0)
-      (effects (font (size 1.27 1.27)) hide)
-    )
-    (property "Part Number" "" (at 330.2 134.62 0)
+    (property "Description" "LED GREEN CLEAR 0603 SMD" (at 330.2 134.62 0)
+      (effects (font (size 1.27 1.27)) hide)
+    )
+    (property "Manufacturer" "Würth Elektronik" (at 330.2 134.62 0)
+      (effects (font (size 1.27 1.27)) hide)
+    )
+    (property "Part Number" "150060VS75000" (at 330.2 134.62 0)
       (effects (font (size 1.27 1.27)) hide)
     )
@@
       (effects (font (size 1.27 1.27)) hide)
     )
-    (property "Datasheet" "~" (at 195.58 187.96 0)
-      (effects (font (size 1.27 1.27)) hide)
-    )
+    (property "Datasheet" "https://cdn.amphenol-cs.com/media/wysiwyg/files/drawing/20021121.pdf" (at 195.58 187.96 0)
+      (effects (font (size 1.27 1.27)) hide)
+    )
+    (property "Description" "CONN HEADER 6 POS 1.27MM VERT" (at 195.58 187.96 0)
+      (effects (font (size 1.27 1.27)) hide)
+    )
+    (property "Manufacturer" "Amphenol ICC (FCI)" (at 195.58 187.96 0)
+      (effects (font (size 1.27 1.27)) hide)
+    )
+    (property "Part Number" "20021121-00006C4LF" (at 195.58 187.96 0)
+      (effects (font (size 1.27 1.27)) hide)
+    )

Commit message: Added P2.0.1
Parts:
- R6: value 20k -> 40k; Part Number RMCF0402FT20K0 -> RMCF0402FT40K2
Changed lines of the file:
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@@
       (effects (font (size 1.27 1.27)) (justify left))
     )
-    (property "Value" "20k" (at 135.89 35.56 0)
+    (property "Value" "40k" (at 135.89 35.56 0)
       (effects (font (size 1.27 1.27)) (justify left))
     )
@@
       (effects (font (size 1.27 1.27)) hide)
     )
-    (property "Description" "RES 20k OHM 1/16W 1% 0402 SMD" (at 133.35 34.29 0)
+    (property "Description" "RES 40.2k OHM 1/16W 1% 0402 SMD" (at 133.35 34.29 0)
       (effects (font (size 1.27 1.27)) hide)
     )
@@
       (effects (font (size 1.27 1.27)) hide)
     )
-    (property "Part Number" "RMCF0402FT20K0" (at 133.35 34.29 0)
+    (property "Part Number" "RMCF0402FT40K2" (at 133.35 34.29 0)
       (effects (font (size 1.27 1.27)) hide)
     )

Commit message: Design review updates
Parts:
- removed R20: 10k, Resistor_SMD:R_0402_1005Metric, symbol Device:R
- C24, C25: value 1uF -> 0.1uF; Part Number C1005X5R1E105K050BC -> C1005X7R1C104K050BC
Connections:
- net STAGE_3_OUT: now also U5.4 (P0.02/AIN0)
Changed lines of the file:
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@@
   (junction (at 118.11 45.72) (diameter 0) (color 0 0 0 0)
   )
-  (junction (at 245.11 71.12) (diameter 0) (color 0 0 0 0)
-  )
   (junction (at 250.19 129.54) (diameter 0) (color 0 0 0 0)
   )
@@
     (stroke (width 0) (type default))
   )
-  (wire (pts (xy 45.085 133.35) (xy 47.625 133.35))
+  (wire (pts (xy 32.385 133.35) (xy 47.625 133.35))
     (stroke (width 0) (type default))
   )
@@
     (stroke (width 0) (type default))
   )
-  (wire (pts (xy 245.11 45.72) (xy 245.11 71.12))
+  (wire (pts (xy 247.65 45.72) (xy 247.65 71.12))
     (stroke (width 0) (type default))
   )
@@
     (stroke (width 0) (type default))
   )
-  (wire (pts (xy 171.45 45.72) (xy 245.11 45.72))
+  (wire (pts (xy 171.45 45.72) (xy 247.65 45.72))
     (stroke (width 0) (type default))
   )
@@
     (stroke (width 0) (type default))
   )
-  (wire (pts (xy 245.11 71.12) (xy 247.65 71.12))
-    (stroke (width 0) (type default))
-  )
   (wire (pts (xy 92.71 57.785) (xy 97.79 57.785))
     (stroke (width 0) (type default))
@@
     (stroke (width 0) (type default))
   )
+  (wire (pts (xy 242.57 71.12) (xy 247.65 71.12))
+    (stroke (width 0) (type default))
+  )
   (wire (pts (xy 189.23 43.18) (xy 265.43 43.18))
     (stroke (width 0) (type default))
@@
     (stroke (width 0) (type default))
   )
-  (wire (pts (xy 32.385 133.35) (xy 37.465 133.35))
-    (stroke (width 0) (type default))
-  )
   (wire (pts (xy 171.45 43.18) (xy 179.07 43.18))
     (stroke (width 0) (type default))
@@
     (stroke (width 0) (type default))
   )
-  (wire (pts (xy 242.57 71.12) (xy 245.11 71.12))
-    (stroke (width 0) (type default))
-  )
   (wire (pts (xy 248.92 129.54) (xy 250.19 129.54))
     (stroke (width 0) (type default))
@@
     (stroke (width 0) (type default))
   )
+  (wire (pts (xy 177.165 27.94) (xy 180.34 27.94))
+    (stroke (width 0) (type default))
+  )
   (wire (pts (xy 232.41 125.73) (xy 219.71 125.73))
     (stroke (width 0) (type default))
@@
   )
   (symbol (lib_id "My_Library:TLV9102") (at 162.56 40.64 0) (unit 1)
-    (in_bom yes) (on_board yes) (dnp no) (fields_autoplaced)
-    (property "Reference" "U2" (at 163.195 36.83 0)
+    (in_bom yes) (on_board yes) (dnp no)
+    (property "Reference" "U2" (at 163.195 36.195 0)
       (effects (font (size 1.27 1.27)))
     )
@@
     )
   )
-  (symbol (lib_id "Device:R") (at 41.275 133.35 90) (unit 1)
-    (in_bom yes) (on_board yes) (dnp no)
-    (property "Reference" "R20" (at 41.275 137.16 90)
-      (effects (font (size 1.27 1.27)))
-    )
-    (property "Value" "10k" (at 41.275 139.7 90)
-      (effects (font (size 1.27 1.27)))
-    )
-    (property "Footprint" "Resistor_SMD:R_0402_1005Metric" (at 41.275 135.128 90)
-      (effects (font (size 1.27 1.27)) hide)
-    )
-    (property "Datasheet" "https://www.seielect.com/catalog/sei-rmcf_rmcp.pdf" (at 41.275 133.35 0)
-      (effects (font (size 1.27 1.27)) hide)
-    )
-    (property "Description" "RES 10k OHM 1/16W 1% 0402 SMD" (at 41.275 133.35 0)
-      (effects (font (size 1.27 1.27)) hide)
-    )
-    (property "Manufacturer" "Stackpole Electronics Inc" (at 41.275 133.35 0)
-      (effects (font (size 1.27 1.27)) hide)
-    )
-    (property "Part Number" "RMCF0402FT10K0" (at 41.275 133.35 0)
-      (effects (font (size 1.27 1.27)) hide)
-    )
-    (pin "2")
-    (pin "1")
-    (instances
-      (project "P2.0"
-        (path "/cc4d5c34-4776-48f9-a8ce-15f2c8e358ac"
-          (reference "R20") (unit 1)
-        )
-      )
-    )
-  )
   (symbol (lib_id "power:+3V3") (at 97.79 24.765 0) (unit 1)
     (in_bom yes) (on_board yes) (dnp no) (fields_autoplaced)
@@
     )
   )
-  (symbol (lib_id "power:GND") (at 180.34 27.94 180) (unit 1)
-    (in_bom yes) (on_board yes) (dnp no) (fields_autoplaced)
-    (property "Reference" "#PWR029" (at 180.34 21.59 0)
+  (symbol (lib_id "power:GND") (at 177.165 27.94 0) (unit 1)
+    (in_bom yes) (on_board yes) (dnp no)
+    (property "Reference" "#PWR029" (at 177.165 34.29 0)
       (effects (font (size 1.27 1.27)) hide)
     )
-    (property "Value" "GND" (at 180.34 22.86 0)
-      (effects (font (size 1.27 1.27)))
+    (property "Value" "GND" (at 171.45 29.21 0)
+      (effects (font (size 1.27 1.27)) (justify left))
     )
-    (property "Footprint" "" (at 180.34 27.94 0)
+    (property "Footprint" "" (at 177.165 27.94 0)
       (effects (font (size 1.27 1.27)) hide)
     )
-    (property "Datasheet" "" (at 180.34 27.94 0)
+    (property "Datasheet" "" (at 177.165 27.94 0)
       (effects (font (size 1.27 1.27)) hide)
     )
@@
     )
   )
-  (symbol (lib_id "power:GND") (at 97.155 109.22 270) (unit 1)
+  (symbol (lib_id "power:GND") (at 97.155 109.22 0) (unit 1)
     (in_bom yes) (on_board yes) (dnp no)
-    (property "Reference" "#PWR021" (at 90.805 109.22 0)
+    (property "Reference" "#PWR021" (at 97.155 115.57 0)
       (effects (font (size 1.27 1.27)) hide)
     )
-    (property "Value" "GND" (at 92.075 109.22 90)
+    (property "Value" "GND" (at 97.155 114.3 0)
       (effects (font (size 1.27 1.27)))
     )
@@
       (effects (font (size 1.27 1.27)) (justify right))
     )
-    (property "Value" "1uF" (at 152.4 54.61 0)
+    (property "Value" "0.1uF" (at 152.4 54.61 0)
       (effects (font (size 1.27 1.27)) (justify right))
     )
@@
       (effects (font (size 1.27 1.27)) hide)
     )
-    (property "Description" "CAP CER 1uF 25V 10% 0402 SMD" (at 148.59 53.34 0)
+    (property "Description" "CAP CER 0.1uF 16V 10% 0402 SMD" (at 148.59 53.34 0)
       (effects (font (size 1.27 1.27)) hide)
     )
@@
       (effects (font (size 1.27 1.27)) hide)
     )
-    (property "Part Number" "C1005X5R1E105K050BC" (at 148.59 53.34 0)
+    (property "Part Number" "C1005X7R1C104K050BC" (at 148.59 53.34 0)
       (effects (font (size 1.27 1.27)) hide)
     )
@@
       (effects (font (size 1.27 1.27)) (justify left))
     )
-    (property "Value" "1uF" (at 184.15 35.56 0)
+    (property "Value" "0.1uF" (at 184.15 35.56 0)
       (effects (font (size 1.27 1.27)) (justify left))
     )
@@
       (effects (font (size 1.27 1.27)) hide)
     )
-    (property "Description" "CAP CER 1uF 25V 10% 0402 SMD" (at 180.34 34.29 0)
+    (property "Description" "CAP CER 0.1uF 16V 10% 0402 SMD" (at 180.34 34.29 0)
       (effects (font (size 1.27 1.27)) hide)
     )
@@
       (effects (font (size 1.27 1.27)) hide)
     )
-    (property "Part Number" "C1005X5R1E105K050BC" (at 180.34 34.29 0)
+    (property "Part Number" "C1005X7R1C104K050BC" (at 180.34 34.29 0)
       (effects (font (size 1.27 1.27)) hide)
     )
