File: PCB_design_files/P2.0.1/P2.0.kicad_pcb (KiCad board)
At the start: 4 copper layers, 19.8 x 19.5 mm, 58 parts, among them J1 EEG_IN, J2 Conn_02x03_Counter_Clockwise, U1 INA819IDRGR, U2 TLV9102IDSGR, U3 TPS61094, U4 TPS60400, U5 NRF52832-QFAA-R, Y1 32MHz

Commit message: Add media files for project submission
Parts:
- removed R20: 10k, Resistor_SMD:R_0402_1005Metric
- C24, C25: value 1uF -> 0.1uF
- R6: value 20k -> 40k
- moved C23 0.41 mm to (85.0, 52.4)
- moved R1 0.25 mm to (81.3, 56.2)
- moved R3 0.20 mm to (80.1, 54.9)
- moved U1 0.20 mm to (84.0, 54.9)
- moved R2 0.15 mm to (81.3, 53.5)
Connections:
- U5 pad 4: Net-(U5-P0.02/AIN0) -> STAGE_3_OUT
Routing:
- net STAGE_3_OUT: track 3.32 -> 5.08 mm
- net GND: track 48.8 -> 50.2 mm, vias 31 -> 30
- net Net-(U5-P0.02/AIN0): track 1.35 -> 0.00 mm
- net -3V3: track 50.8 -> 51.8 mm
- net /EEG-: track 8.10 -> 7.12 mm
